File: Ebi Cap Charger.kicad_sch (KiCad schematic)
At the start: 1 part

Commit message: Started schematic
Parts:
- removed U?: LT3748xMS, Package_SO:Linear_MSOP-12-16_3x4mm_P0.5mm, symbol Regulator_Switching:LT3748xMS
- added Q? (x3): FET, symbol Device:Q_NMOS_GDS
- added R? (x6): 0R01, symbol Device:R
- added R?: 787R, symbol Device:R
- added R? (x6): 100K, symbol Device:R
- added R?: 18K2, symbol Device:R
- added R? (x2): 40K2, symbol Device:R
- added U?: LT3751, SOP65P640X120-21N, symbol LT3751:LT3751IFEPBF
Connections:
- new net: Q?.3 (S), Q?.3 (S), R?.1, R?.1, R?.1, R?.1, R?.1, R?.1, U?.12 (CSP)
- new net: R?.1, U?.16 (RBG)
- new net: R?.1, R?.1, R?.1, R?.1, R?.1, R?.1, R?.2, U?.13 (VCC), U?.14 (LVGATE)
- new net: R?.2, U?.6 (~{FAULT})
- new net: Q?.1 (G), Q?.1 (G), Q?.1 (G), U?.15 (HVGATE)
- new net: Q?.2 (D), Q?.2 (D), Q?.2 (D), R?.2, R?.2
- new net: R?.2, U?.3 (OVLO1)
- new net: R?.2, U?.7 (~{DONE})
- new net: R?.1, U?.20 (RDCM)
- new net: R?.2, U?.2 (UVLO1)
- new net: R?.2, U?.4 (UVLO2)
- new net: R?.2, U?.5 (OVLO2)
- new net: R?.1, U?.1 (RVTRANS)
- new net: R?.1, U?.18 (RVOUT)
- new net GND: R?.2, R?.2, R?.2, R?.2, R?.2, R?.2, R?.2, U?.10 (FB), U?.11 (CSN), U?.21 (GND), U?.9 (CLAMP)

Commit message: updated PCB
Parts:
- removed Q?: FET, symbol Device:Q_NMOS_GDS
- removed R? (x2): 0R01, symbol Device:R
- added C1, C2, C3: 1uF, Capacitor_SMD:C_1206_3216Metric, symbol Device:C_Small
- added C4, C5, C6, C7: 100uF, Capacitor_SMD:C_2220_5650Metric, symbol Device:C_Small
- added D1, D2, D3: D, Diode_SMD:D_SMB, symbol Device:D
- added U2, U3, U4: DA2034-AL, DA2034:DA2034-AL, symbol DA2034:DA2034-AL
- Q1, Q2: renamed from Q?; footprint (none) -> Package_TO_SOT_SMD:TO-252-2
- R1, R10, R2, R3, R4, R5, R6, R7, R8, R9: renamed from R?; footprint (none) -> Resistor_SMD:R_0603_1608Metric
- R11, R12, R13, R14: renamed from R?; footprint (none) -> Resistor_SMD:R_2512_6332Metric
- U1: renamed from U?; footprint SOP65P640X120-21N -> Package_SO:TSSOP-20_4.4x6.5mm_P0.65mm
Connections:
- net GND: now also C4.2, C5.2, C6.2, C7.2
- net at R1.1, R2.1, R3.1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: now also C4.1, C5.1, C6.1, C7.1, U2.P$3, U2.P$4, U2.P$5, U2.P$6, U3.P$3, U3.P$4, U3.P$5, U3.P$6, U4.P$3, U4.P$4, U4.P$5, U4.P$6
- net at Q1.2 (D), Q2.2 (D), R10.2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: now also U2.P$10, U2.P$7, U2.P$8, U2.P$9, U3.P$10, U3.P$7, U3.P$8, U3.P$9, U4.P$10, U4.P$7, U4.P$8, U4.P$9
- new net: C1.1, D1.1 (K)
- new net: D1.2 (A), U2.P$12
- new net: C2.2, U3.P$1
- new net: D2.2 (A), U3.P$12
- new net: C3.2, U4.P$1
- new net: D3.2 (A), U4.P$12
- new net: C2.1, D2.1 (K)
- new net: C1.2, U2.P$1
- new net: C3.1, D3.1 (K)
Other:
- moved on the sheet: Q1, Q2, R1, R10, R11, R12, R13, R14, R2, R3, R4, R5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

Commit message: updated PCB
Parts:
- added C8: 10uF, Capacitor_SMD:C_0603_1608Metric, symbol Device:C_Small
- U1: footprint Package_SO:TSSOP-20_4.4x6.5mm_P0.65mm -> Package_SO:HTSSOP-20-1EP_4.4x6.5mm_P0.65mm_EP2.74x3.86mm
Connections:
- net GND: now also C8.1
- net at C4.1, C5.1, C6.1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: now also C8.2
Changed lines of the file:
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@@
+    (stroke (width 0) (type default) (color 0 0 0 0))
+  )
+  (wire (pts (xy 40.64 149.86) (xy 40.64 147.32))
     (stroke (width 0) (type default) (color 0 0 0 0))
   )
@@
     (stroke (width 0) (type default) (color 0 0 0 0))
   )
+  (wire (pts (xy 40.64 147.32) (xy 45.72 147.32))
+    (stroke (width 0) (type default) (color 0 0 0 0))
+  )
   (wire (pts (xy 153.67 116.84) (xy 153.67 129.54))
     (stroke (width 0) (type default) (color 0 0 0 0))
@@
   )
   (wire (pts (xy 203.2 132.08) (xy 198.12 132.08))
+    (stroke (width 0) (type default) (color 0 0 0 0))
+  )
+  (wire (pts (xy 40.64 157.48) (xy 40.64 154.94))
     (stroke (width 0) (type default) (color 0 0 0 0))
   )
@@
     (pin "2")
   )
+  (symbol (lib_id "Device:C_Small") (at 40.64 152.4 0) (mirror x) (unit 1)
+    (in_bom yes) (on_board yes) (fields_autoplaced)
+    (property "Reference" "C8" (id 0) (at 38.316 151.4851 0)
+      (effects (font (size 1.27 1.27)) (justify right))
+    )
+    (property "Value" "10uF" (id 1) (at 38.316 154.2602 0)
+      (effects (font (size 1.27 1.27)) (justify right))
+    )
+    (property "Footprint" "Capacitor_SMD:C_0603_1608Metric" (id 2) (at 40.64 152.4 0)
+      (effects (font (size 1.27 1.27)) hide)
+    )
+    (property "Datasheet" "~" (id 3) (at 40.64 152.4 0)
+      (effects (font (size 1.27 1.27)) hide)
+    )
+    (pin "1")
+    (pin "2")
+  )
   (symbol (lib_id "Device:R") (at 52.07 163.83 90) (unit 1)
     (in_bom yes) (on_board yes)
@@
     (pin "1")
     (pin "2")
+  )
+  (symbol (lib_id "power:GND") (at 40.64 157.48 0) (unit 1)
+    (in_bom yes) (on_board yes) (fields_autoplaced)
+    (property "Reference" "#PWR03" (id 0) (at 40.64 163.83 0)
+      (effects (font (size 1.27 1.27)) hide)
+    )
+    (property "Value" "GND" (id 1) (at 40.64 162.0425 0))
+    (property "Footprint" "" (id 2) (at 40.64 157.48 0)
+      (effects (font (size 1.27 1.27)) hide)
+    )
+    (property "Datasheet" "" (id 3) (at 40.64 157.48 0)
+      (effects (font (size 1.27 1.27)) hide)
+    )
+    (pin "1")
   )
   (symbol (lib_id "Device:R") (at 127 171.45 0) (unit 1)
@@
       (effects (font (size 1.27 1.27)) (justify left))
     )
-    (property "Footprint" "Package_SO:TSSOP-20_4.4x6.5mm_P0.65mm" (id 2) (at 63.5 210.82 0)
+    (property "Footprint" "Package_SO:HTSSOP-20-1EP_4.4x6.5mm_P0.65mm_EP2.74x3.86mm" (id 2) (at 63.5 210.82 0)
       (effects (font (size 1.27 1.27)) (justify left bottom) hide)
     )
@@
       (reference "#PWR02") (unit 1) (value "GND") (footprint "")
     )
+    (path "/6f8fbbf9-fc22-4814-861b-3cc4e37d9a53"
+      (reference "#PWR03") (unit 1) (value "GND") (footprint "")
+    )
     (path "/d4ba7d3e-baad-4a0d-bcee-4c54e56b670a"
       (reference "#PWR0101") (unit 1) (value "GND") (footprint "")
@@
       (reference "C7") (unit 1) (value "100uF") (footprint "Capacitor_SMD:C_2220_5650Metric")
     )
+    (path "/58d93802-f702-40b7-8cde-c973c90469df"
+      (reference "C8") (unit 1) (value "10uF") (footprint "Capacitor_SMD:C_0603_1608Metric")
+    )
     (path "/19fa455b-e8f9-4a71-a821-82149399eb2e"
       (reference "D1") (unit 1) (value "D") (footprint "Diode_SMD:D_SMB")
@@
     )
     (path "/d03e8b8e-d22c-4974-b7de-91c177947b0a"
-      (reference "U1") (unit 1) (value "LT3751") (footprint "Package_SO:TSSOP-20_4.4x6.5mm_P0.65mm")
+      (reference "U1") (unit 1) (value "LT3751") (footprint "Package_SO:HTSSOP-20-1EP_4.4x6.5mm_P0.65mm_EP2.74x3.86mm")
     )
     (path "/b37ba0e4-c660-44d5-bd24-47ff6d2ba9c7"

Commit message: Updated PCB
Changed lines of the file:
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@@
   (junction (at 45.72 156.21) (diameter 0) (color 0 0 0 0)
   )
+  (junction (at 104.14 167.64) (diameter 0) (color 0 0 0 0)
+  )
   (junction (at 45.72 152.4) (diameter 0) (color 0 0 0 0)
   )
@@
   (junction (at 104.14 165.1) (diameter 0) (color 0 0 0 0)
   )
+  (junction (at 104.14 175.26) (diameter 0) (color 0 0 0 0)
+  )
   (junction (at 104.14 149.86) (diameter 0) (color 0 0 0 0)
   )
@@
     (stroke (width 0) (type default) (color 0 0 0 0))
   )
+  (wire (pts (xy 91.44 177.8) (xy 101.6 177.8))
+    (stroke (width 0) (type default) (color 0 0 0 0))
+  )
   (wire (pts (xy 104.14 93.98) (xy 109.22 93.98))
     (stroke (width 0) (type default) (color 0 0 0 0))
@@
     (stroke (width 0) (type default) (color 0 0 0 0))
   )
-  (wire (pts (xy 91.44 177.8) (xy 104.14 177.8))
-    (stroke (width 0) (type default) (color 0 0 0 0))
-  )
   (wire (pts (xy 48.26 156.21) (xy 45.72 156.21))
     (stroke (width 0) (type default) (color 0 0 0 0))
@@
     (stroke (width 0) (type default) (color 0 0 0 0))
   )
+  (wire (pts (xy 91.44 165.1) (xy 101.6 165.1))
+    (stroke (width 0) (type default) (color 0 0 0 0))
+  )
   (wire (pts (xy 45.72 167.64) (xy 45.72 171.45))
     (stroke (width 0) (type default) (color 0 0 0 0))
@@
     (stroke (width 0) (type default) (color 0 0 0 0))
   )
-  (wire (pts (xy 91.44 165.1) (xy 104.14 165.1))
-    (stroke (width 0) (type default) (color 0 0 0 0))
-  )
   (wire (pts (xy 151.13 119.38) (xy 151.13 132.08))
     (stroke (width 0) (type default) (color 0 0 0 0))
@@
     (stroke (width 0) (type default) (color 0 0 0 0))
   )
+  (wire (pts (xy 101.6 165.1) (xy 104.14 167.64))
+    (stroke (width 0) (type default) (color 0 0 0 0))
+  )
   (wire (pts (xy 45.72 152.4) (xy 45.72 156.21))
     (stroke (width 0) (type default) (color 0 0 0 0))
   )
+  (wire (pts (xy 104.14 175.26) (xy 101.6 177.8))
+    (stroke (width 0) (type default) (color 0 0 0 0))
+  )

Commit message: Updated PCB
Parts:
- removed C4: 100uF, Capacitor_SMD:C_2220_5650Metric, symbol Device:C_Small
- C5, C6: value 100uF -> 470uF; footprint Capacitor_SMD:C_2220_5650Metric -> Capacitor_THT:CP_Radial_D10.0mm_P5.00mm
Changed lines of the file:
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@@
   (junction (at 45.72 160.02) (diameter 0) (color 0 0 0 0)
   )
-  (junction (at 45.72 100.33) (diameter 0) (color 0 0 0 0)
-  )
   (junction (at 119.38 177.8) (diameter 0) (color 0 0 0 0)
   )
@@
   (junction (at 106.68 116.84) (diameter 0) (color 0 0 0 0)
   )
-  (junction (at 57.15 88.9) (diameter 0) (color 0 0 0 0)
-  )
   (junction (at 104.14 165.1) (diameter 0) (color 0 0 0 0)
   )
@@
     (stroke (width 0) (type default) (color 0 0 0 0))
   )
-  (wire (pts (xy 57.15 92.71) (xy 57.15 88.9))
-    (stroke (width 0) (type default) (color 0 0 0 0))
-  )
   (wire (pts (xy 198.12 119.38) (xy 203.2 119.38))
     (stroke (width 0) (type default) (color 0 0 0 0))
@@
     (stroke (width 0) (type default) (color 0 0 0 0))
   )
-  (wire (pts (xy 45.72 100.33) (xy 57.15 100.33))
-    (stroke (width 0) (type default) (color 0 0 0 0))
-  )
-  (wire (pts (xy 57.15 97.79) (xy 57.15 100.33))
-    (stroke (width 0) (type default) (color 0 0 0 0))
-  )
   (wire (pts (xy 101.6 165.1) (xy 104.14 167.64))
     (stroke (width 0) (type default) (color 0 0 0 0))
@@
     (stroke (width 0) (type default) (color 0 0 0 0))
   )
-  (wire (pts (xy 45.72 88.9) (xy 57.15 88.9))
+  (wire (pts (xy 45.72 88.9) (xy 73.66 88.9))
     (stroke (width 0) (type default) (color 0 0 0 0))
   )
@@
   )
   (wire (pts (xy 104.14 147.32) (xy 104.14 149.86))
-    (stroke (width 0) (type default) (color 0 0 0 0))
-  )
-  (wire (pts (xy 57.15 88.9) (xy 73.66 88.9))
     (stroke (width 0) (type default) (color 0 0 0 0))
   )
@@
       (effects (font (size 1.27 1.27)) (justify left))
     )
-    (property "Value" "100uF" (id 1) (at 36.6141 97.1229 0)
-      (effects (font (size 1.27 1.27)) (justify left))
-    )
-    (property "Footprint" "Capacitor_SMD:C_2220_5650Metric" (id 2) (at 34.29 95.25 0)
+    (property "Value" "470uF" (id 1) (at 36.6141 97.1229 0)
+      (effects (font (size 1.27 1.27)) (justify left))
+    )
+    (property "Footprint" "Capacitor_THT:CP_Radial_D10.0mm_P5.00mm" (id 2) (at 34.29 95.25 0)
       (effects (font (size 1.27 1.27)) hide)
     )
@@
     (pin "P$9")
   )
-  (symbol (lib_id "Device:C_Small") (at 57.15 95.25 0) (unit 1)
-    (in_bom yes) (on_board yes) (fields_autoplaced)
-    (property "Reference" "C4" (id 0) (at 59.4741 94.3478 0)
-      (effects (font (size 1.27 1.27)) (justify left))
-    )
-    (property "Value" "100uF" (id 1) (at 59.4741 97.1229 0)
-      (effects (font (size 1.27 1.27)) (justify left))
-    )
-    (property "Footprint" "Capacitor_SMD:C_2220_5650Metric" (id 2) (at 57.15 95.25 0)
-      (effects (font (size 1.27 1.27)) hide)
-    )
-    (property "Datasheet" "~" (id 3) (at 57.15 95.25 0)
-      (effects (font (size 1.27 1.27)) hide)
-    )
-    (pin "1")
-    (pin "2")
-  )
   (symbol (lib_id "Device:R") (at 52.07 171.45 90) (unit 1)
     (in_bom yes) (on_board yes)
@@
       (effects (font (size 1.27 1.27)) (justify left))
     )
-    (property "Value" "100uF" (id 1) (at 25.1841 97.1229 0)
-      (effects (font (size 1.27 1.27)) (justify left))
-    )
-    (property "Footprint" "Capacitor_SMD:C_2220_5650Metric" (id 2) (at 22.86 95.25 0)
+    (property "Value" "470uF" (id 1) (at 25.1841 97.1229 0)
+      (effects (font (size 1.27 1.27)) (justify left))
+    )
+    (property "Footprint" "Capacitor_THT:CP_Radial_D10.0mm_P5.00mm" (id 2) (at 22.86 95.25 0)
       (effects (font (size 1.27 1.27)) hide)
     )
@@
       (reference "C3") (unit 1) (value "1uF") (footprint "Capacitor_SMD:C_1206_3216Metric")
     )
-    (path "/b9aa6545-b6a4-4f83-8c21-74599078fd25"
-      (reference "C4") (unit 1) (value "100uF") (footprint "Capacitor_SMD:C_2220_5650Metric")
-    )
     (path "/ecdc0307-8a49-4ea1-936e-d70fe3f9f6e9"
-      (reference "C5") (unit 1) (value "100uF") (footprint "Capacitor_SMD:C_2220_5650Metric")
+      (reference "C5") (unit 1) (value "470uF") (footprint "Capacitor_THT:CP_Radial_D10.0mm_P5.00mm")
     )
     (path "/8e9c6039-69c1-4531-8225-a289ab5e1c73"
-      (reference "C6") (unit 1) (value "100uF") (footprint "Capacitor_SMD:C_2220_5650Metric")
+      (reference "C6") (unit 1) (value "470uF") (footprint "Capacitor_THT:CP_Radial_D10.0mm_P5.00mm")
     )
     (path "/8f3ffd16-dbbe-4aa3-bf22-82d6dbbc92cf"

Commit message: PCB draft
Parts:
- added H1, H2, H3, H4: MountingHole, MountingHole:MountingHole_3.2mm_M3_Pad_Via, symbol Mechanical:MountingHole
- added J1: VIN, Connector_PinHeader_2.54mm:PinHeader_1x02_P2.54mm_Vertical, symbol Connector_Generic:Conn_01x02
- added J2: C1, Connector_PinHeader_2.54mm:PinHeader_1x02_P2.54mm_Vertical, symbol Connector_Generic:Conn_01x02
- added J3: C2, Connector_PinHeader_2.54mm:PinHeader_1x02_P2.54mm_Vertical, symbol Connector_Generic:Conn_01x02
- added J4: C3, Connector_PinHeader_2.54mm:PinHeader_1x02_P2.54mm_Vertical, symbol Connector_Generic:Conn_01x02
Connections:
- net GND: now also J1.2 (Pin_2)
- net at C1.1, D1.1 (K): now also J2.1 (Pin_1)
- net at C5.1, C6.1, C7.1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: now also J1.1 (Pin_1)
- net at C2.2, U3.P$1: now also J3.2 (Pin_2)
- net at C3.2, U4.P$1: now also J4.2 (Pin_2)
- net at C2.1, D2.1 (K): now also J3.1 (Pin_1)
- net at C1.2, U2.P$1: now also J2.2 (Pin_2)
- net at C3.1, D3.1 (K): now also J4.1 (Pin_1)
Other:
- moved on the sheet: C1, C2, C3, C5, C6, C7, C8, D1, D2, D3, Q1, Q2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
